Commit message: added dvl and localization

File: mini_alpha_description/urdf/base.urdf (robot description, URDF)
Before this commit: robot mini_alpha, 11 links, 10 joints
Links:
- added link dvl
Joints:
- added joint dvl_joint: type fixed, parent base_link, child dvl, origin xyz=-0.1 0.0 -0.1 rpy=0.0 0.0 0.0
